Commit message: Progress!

File: nav2_min_tb4_description/urdf/icreate/common_properties.urdf.xacro (robot description, xacro)
@@ -49,5 +49,5 @@
       <visualize>${visualize}</visualize>
       <always_on>true</always_on>
-      <gz_frame_id>base_scan</gz_frame_id>
+      <gz_frame_id>${sensor_name}_link</gz_frame_id>
       <topic>scan</topic>
       <lidar>

File: nav2_min_tb4_description/urdf/icreate/wheel.urdf.xacro (robot description, xacro)
@@ -1,5 +1,5 @@
 <?xml version="1.0"?>
 <robot xmlns:xacro="http://ros.org/wiki/xacro">
-<xacro:macro name="wheel" params="name gazebo parent_link *origin">
+<xacro:macro name="wheel" params="name gazebo parent_link:=base_link *origin">
   <xacro:property name="mass"   value="0.2" />
   <xacro:property name="radius" value="${3.575*cm2m}" />
