Commit message: fixing up for use

File: nav2_min_tb4_description/urdf/standard/turtlebot4.urdf.xacro (robot description, xacro)
@@ -38,4 +38,23 @@
     <origin xyz="0 0 ${shell_z_offset + base_link_z_offset}" rpy="0 0 0"/>
   </joint>
+  <!-- Add a base footprint definition -->
+  <joint name="base_footprint_joint" type="fixed">
+    <parent link="base_link"/>
+    <child link="base_footprint"/>
+    <origin xyz="0 0 0" rpy="0 0 0"/>
+  </joint>
+  <link name="base_footprint">
+    <inertial>
+      <mass value="0.0001"/>
+      <origin xyz="0 0 0"/>
+      <inertia ixx="0.0001" ixy="0.0" ixz="0.0" iyy="0.0001" iyz="0.0" izz="0.0001"/>
+    </inertial>
+    <visual>
+      <origin rpy="0 0 0" xyz="0 0 0"/>
+      <geometry>
+        <box size="0.001 0.001 0.001"/>
+      </geometry>
+    </visual>
+  </link>
   <!-- Turtlebot4 shell definition -->
   <link name="shell_link">
