Commit message: feat(sensor): add 3d lidar veloyne
Signed-off-by: elsayed <elsayed.elsheikh97@gmail.com>

File: nav2_minimal_tb4_description/urdf/icreate/common_properties.urdf.xacro (robot description, xacro)
@@ -42,6 +42,7 @@
   </xacro:macro>
   <xacro:macro name="ray_sensor"
-    params="sensor_name gazebo update_rate visualize
+    params="sensor_name use_vertical_rays:=^|false gazebo update_rate visualize
             h_samples h_res h_min_angle h_max_angle
+            v_samples:=^|0 v_res:=^|0 v_min_angle:=^|0 v_max_angle:=^|0
             r_min r_max r_res *plugin">
     <sensor name="${sensor_name}" type="gpu_lidar">
@@ -59,4 +60,12 @@
             <max_angle>${h_max_angle}</max_angle>
           </horizontal>
+          <xacro:if value="${use_vertical_rays}">
+            <vertical>
+              <samples>${v_samples}</samples>
+              <resolution>${v_res}</resolution>
+              <min_angle>${v_min_angle}</min_angle>
+              <max_angle>${v_max_angle}</max_angle>
+            </vertical>
+          </xacro:if>
         </scan>
         <range>

File: nav2_minimal_tb4_description/urdf/standard/turtlebot4.urdf.xacro (robot description, xacro)
@@ -4,4 +4,5 @@
   <xacro:include filename="$(find nav2_minimal_tb4_description)/urdf/icreate/create3.urdf.xacro" />
   <xacro:include filename="$(find nav2_minimal_tb4_description)/urdf/sensors/rplidar.urdf.xacro" />
+  <xacro:include filename="$(find nav2_minimal_tb4_description)/urdf/sensors/velodyne.urdf.xacro" />
   <xacro:include filename="$(find nav2_minimal_tb4_description)/urdf/sensors/oakd.urdf.xacro" />
   <xacro:include filename="$(find nav2_minimal_tb4_description)/urdf/sensors/camera_bracket.urdf.xacro" />
@@ -110,8 +111,17 @@
   </xacro:tower_sensor_plate>
   <!-- Turtlebot4 sensor definitions -->
-  <xacro:rplidar name="rplidar" parent_link="shell_link" gazebo="$(arg gazebo)">
-    <origin xyz="${rplidar_x_offset} ${rplidar_y_offset} ${rplidar_z_offset}"
-            rpy="0 0 ${pi/2}"/>
-  </xacro:rplidar>
+  <xacro:arg name="use_3d_lidar" default="false" />
+  <xacro:unless value="$(arg use_3d_lidar)">
+    <xacro:rplidar name="rplidar" parent_link="shell_link" gazebo="$(arg gazebo)">
+      <origin xyz="${rplidar_x_offset} ${rplidar_y_offset} ${rplidar_z_offset}"
+              rpy="0 0 ${pi/2}"/>
+    </xacro:rplidar>
+  </xacro:unless>
+  <xacro:if value="$(arg use_3d_lidar)">
+    <xacro:velodyne name="velodyne" parent_link="shell_link" gazebo="$(arg gazebo)">
+      <origin xyz="${rplidar_x_offset} ${rplidar_y_offset} ${rplidar_z_offset}"
+              rpy="0 0 ${pi/2}"/>
+    </xacro:velodyne>
+  </xacro:if>
   <xacro:camera_bracket name="oakd_camera_bracket">
     <origin xyz="${camera_mount_x_offset} ${camera_mount_y_offset} ${camera_mount_z_offset}"/>
