Commit message: Fix missing imu_joint in gz_waffle.sdf.xacro
Signed-off-by: Jabee7531 <jabee7531@gmail.com>

File: nav2_minimal_tb3_sim/urdf/gz_waffle.sdf.xacro (robot description, xacro)
@@ -424,4 +424,9 @@
         </axis>
       </joint>
+      <joint name="imu_joint" type="fixed">
+        <parent>base_link</parent>
+        <child>imu_link</child>
+        <pose>0.0 0 0.068 0 0 0</pose>
+      </joint>
       <plugin
         filename="gz-sim-diff-drive-system"
