Commit message: working version
Signed-off-by: stevedan <stevedan.o.omodolor@gmail.com>

File: nav2_minimal_tb3_sim/urdf/gz_waffle_gps.sdf.xacro (robot description, xacro)
@@ -43,5 +43,5 @@
           <always_on>true</always_on>
           <update_rate>200</update_rate>
-          <topic>$(arg namespace)/imu</topic>
+          <topic>$(arg namespace)/imu/data</topic>
           <gz_frame_id>imu_link</gz_frame_id>
           <imu>
@@ -89,10 +89,10 @@
         </sensor>
       </link>
-      <link name="navsat_link">
+      <link name="gps_link">
         <sensor name="navsat" type="navsat">
           <always_on>true</always_on>
           <update_rate>1</update_rate>
-          <topic>$(arg namespace)/navsat</topic>
-          <pose>0 0 0 0 0 0</pose>
+          <topic>$(arg namespace)/gps/fix</topic>
+          <gz_frame_id>gps_link</gz_frame_id>
           <navsat>
             <position_sensing>
@@ -100,5 +100,5 @@
                 <noise type="gaussian">
                   <mean>0.0</mean>
-                  <stddev>0.1</stddev>
+                  <stddev>0.0</stddev>
                 </noise>
               </horizontal>
@@ -448,4 +448,14 @@
         </axis>
       </joint>
+      <joint name="imu_joint" type="fixed">
+        <parent>base_link</parent>
+        <child>imu_link</child>
+        <pose>0.0 0 0.068 0 0 0</pose>
+      </joint>
+      <joint name="gps_joint" type="fixed">
+        <parent>base_link</parent>
+        <child>gps_link</child>
+        <pose>-0.05 0 0.05 0 0 0</pose>
+      </joint>
       <plugin
         filename="gz-sim-diff-drive-system"

Commit message: use bullet
Signed-off-by: Stevedan Omodolor <stevedan.o.omodolor@gmail.com>

File: nav2_minimal_tb3_sim/urdf/gz_waffle_gps.sdf.xacro (robot description, xacro)
@@ -201,5 +201,5 @@
           <surface>
             <friction>
-              <ode>
+              <bullet>
                 <mu>1</mu>
                 <mu2>1</mu2>
@@ -207,8 +207,8 @@
                 <slip2>0</slip2>
                 <fdir1>0 0 1</fdir1>
-              </ode>
+              </bullet>
             </friction>
             <contact>
-              <ode>
+              <bullet>
                 <soft_cfm>0</soft_cfm>
                 <soft_erp>0.2</soft_erp>
@@ -217,5 +217,5 @@
                 <max_vel>0.01</max_vel>
                 <min_depth>0.001</min_depth>
-              </ode>
+              </bullet>
             </contact>
           </surface>
@@ -257,5 +257,5 @@
           <surface>
             <friction>
-              <ode>
+              <bullet>
                 <mu>1</mu>
                 <mu2>1</mu2>
@@ -263,8 +263,8 @@
                 <slip2>0</slip2>
                 <fdir1>0 0 1</fdir1>
-              </ode>
+              </bullet>
             </friction>
             <contact>
-              <ode>
+              <bullet>
                 <soft_cfm>0</soft_cfm>
                 <soft_erp>0.2</soft_erp>
@@ -273,5 +273,5 @@
                 <max_vel>0.01</max_vel>
                 <min_depth>0.001</min_depth>
-              </ode>
+              </bullet>
             </contact>
           </surface>
@@ -291,5 +291,5 @@
       </link>
       <link name='caster_back_right_link'>
-        <pose>-0.177 -0.064 -0.004 0 0 0</pose>
+        <pose>-0.177 -0.064 -0.004 -1.57 0 0</pose>
         <inertial>
           <mass>0.001</mass>
@@ -303,13 +303,22 @@
           </inertia>
         </inertial>
-        <collision name='collision'>
+        <collision name='caster_back_right_collision'>
           <geometry>
             <sphere>
-              <radius>0.005000</radius>
+              <radius>0.0060000</radius>
             </sphere>
           </geometry>
           <surface>
+            <friction>
+              <bullet>
+                <mu>1</mu>
+                <mu2>1</mu2>
+                <slip1>0.035</slip1>
+                <slip2>0</slip2>
+                <fdir1>0 0 1</fdir1>
+              </bullet>
+            </friction>
             <contact>
-              <ode>
+              <bullet>
                 <soft_cfm>0</soft_cfm>
                 <soft_erp>0.2</soft_erp>
@@ -318,11 +327,23 @@
                 <max_vel>0.01</max_vel>
                 <min_depth>0.001</min_depth>
-              </ode>
+              </bullet>
             </contact>
           </surface>
         </collision>
+        <visual name="sphere_visual">
+          <geometry>
+            <sphere>
+              <radius>0.0060000</radius>
+            </sphere>
+          </geometry>
+          <material>
+            <ambient>0 0 1 1</ambient>
+            <diffuse>0 0 1 1</diffuse>
+            <specular>0 0 1 1</specular>
+          </material>
+        </visual>
       </link>
       <link name='caster_back_left_link'>
-        <pose>-0.177 0.064 -0.004 0 0 0</pose>
+        <pose>-0.177 0.064 -0.004 -1.57 0 0</pose>
         <inertial>
           <mass>0.001</mass>
@@ -336,13 +357,22 @@
           </inertia>
         </inertial>
-        <collision name='collision'>
+        <collision name='caster_back_left_collision'>
           <geometry>
             <sphere>
-              <radius>0.005000</radius>
+              <radius>0.0060000</radius>
             </sphere>
           </geometry>
           <surface>
+            <friction>
+              <bullet>
+                <mu>1</mu>
+                <mu2>1</mu2>
+                <slip1>0.035</slip1>
+                <slip2>0</slip2>
+                <fdir1>0 0 1</fdir1>
+              </bullet>
+            </friction>
             <contact>
-              <ode>
+              <bullet>
                 <soft_cfm>0</soft_cfm>
                 <soft_erp>0.2</soft_erp>
@@ -351,10 +381,23 @@
                 <max_vel>0.01</max_vel>
                 <min_depth>0.001</min_depth>
-              </ode>
+              </bullet>
             </contact>
           </surface>
         </collision>
+       <visual name="sphere_visual">
+          <geometry>
+            <sphere>
+              <radius>0.0060000</radius>
+            </sphere>
+          </geometry>
+          <material>
+            <ambient>0 0 1 1</ambient>
+            <diffuse>0 0 1 1</diffuse>
+            <specular>0 0 1 1</specular>
+          </material>
+        </visual>
       </link>
       <link name="camera_link">
+        <pose>0.069 -0.047 0.107 0 0 0</pose>
         <inertial>
           <pose>0.069 -0.047 0.107 0 0 0</pose>

Commit message: Straighten robot and minor estetic changes (#33)
* Gps navigation Tutorial update

Signed-off-by: Stevedan Omodolor <stevedan.o.omodolor@gmail.com>

* revert back

Signed-off-by: Stevedan Omodolor <stevedan.o.omodolor@gmail.com>

* use bullet

Signed-off-by: Stevedan Omodolor <stevedan.o.omodolor@gmail.com>

* remove friction

Signed-off-by: Stevedan Omodolor <stevedan.o.omodolor@gmail.com>

* cleanup

Signed-off-by: Stevedan Omodolor <stevedan.o.omodolor@gmail.com>

* remove unwanted pose

Signed-off-by: Stevedan Omodolor <stevedan.o.omodolor@gmail.com>

---------

Signed-off-by: Stevedan Omodolor <stevedan.o.omodolor@gmail.com>

File: nav2_minimal_tb3_sim/urdf/gz_waffle_gps.sdf.xacro (robot description, xacro)
@@ -146,5 +146,5 @@
           </geometry>
           <material>
-            <diffuse>1 1 1</diffuse>
+            <diffuse>0.5 0.5 0.5</diffuse>
           </material>
         </visual>
@@ -201,5 +201,5 @@
           <surface>
             <friction>
-              <ode>
+              <bullet>
                 <mu>1</mu>
                 <mu2>1</mu2>
@@ -207,8 +207,8 @@
                 <slip2>0</slip2>
                 <fdir1>0 0 1</fdir1>
-              </ode>
+              </bullet>
             </friction>
             <contact>
-              <ode>
+              <bullet>
                 <soft_cfm>0</soft_cfm>
                 <soft_erp>0.2</soft_erp>
@@ -217,5 +217,5 @@
                 <max_vel>0.01</max_vel>
                 <min_depth>0.001</min_depth>
-              </ode>
+              </bullet>
             </contact>
           </surface>
@@ -230,5 +230,5 @@
           </geometry>
           <material>
-            <diffuse>1 1 1</diffuse>
+            <diffuse>0.5 0.5 0.5</diffuse>
           </material>
         </visual>
@@ -257,5 +257,5 @@
           <surface>
             <friction>
-              <ode>
+              <bullet>
                 <mu>1</mu>
                 <mu2>1</mu2>
@@ -263,8 +263,8 @@
                 <slip2>0</slip2>
                 <fdir1>0 0 1</fdir1>
-              </ode>
+              </bullet>
             </friction>
             <contact>
-              <ode>
+              <bullet>
                 <soft_cfm>0</soft_cfm>
                 <soft_erp>0.2</soft_erp>
@@ -273,5 +273,5 @@
                 <max_vel>0.01</max_vel>
                 <min_depth>0.001</min_depth>
-              </ode>
+              </bullet>
             </contact>
           </surface>
@@ -286,10 +286,10 @@
           </geometry>
           <material>
-            <diffuse>1 1 1</diffuse>
+            <diffuse>0.5 0.5 0.5</diffuse>
           </material>
         </visual>
       </link>
       <link name='caster_back_right_link'>
-        <pose>-0.177 -0.064 -0.004 0 0 0</pose>
+        <pose>-0.177 -0.064 -0.004 -1.57 0 0</pose>
         <inertial>
           <mass>0.001</mass>
@@ -303,13 +303,13 @@
           </inertia>
         </inertial>
-        <collision name='collision'>
+        <collision name='caster_back_right_collision'>
           <geometry>
             <sphere>
-              <radius>0.005000</radius>
+              <radius>0.0060000</radius>
             </sphere>
           </geometry>
           <surface>
             <contact>
-              <ode>
+              <bullet>
                 <soft_cfm>0</soft_cfm>
                 <soft_erp>0.2</soft_erp>
@@ -318,11 +318,21 @@
                 <max_vel>0.01</max_vel>
                 <min_depth>0.001</min_depth>
-              </ode>
+              </bullet>
             </contact>
           </surface>
         </collision>
+        <visual name="sphere_visual">
+          <geometry>
+            <sphere>
+              <radius>0.0060000</radius>
+            </sphere>
+          </geometry>
+          <material>
+            <diffuse>0.5 0.5 0.5</diffuse>
+          </material>
+        </visual>
       </link>
       <link name='caster_back_left_link'>
-        <pose>-0.177 0.064 -0.004 0 0 0</pose>
+        <pose>-0.177 0.064 -0.004 -1.57 0 0</pose>
         <inertial>
           <mass>0.001</mass>
@@ -336,13 +346,13 @@
           </inertia>
         </inertial>
-        <collision name='collision'>
+        <collision name='caster_back_left_collision'>
           <geometry>
             <sphere>
-              <radius>0.005000</radius>
+              <radius>0.0060000</radius>
             </sphere>
           </geometry>
           <surface>
             <contact>
-              <ode>
+              <bullet>
                 <soft_cfm>0</soft_cfm>
                 <soft_erp>0.2</soft_erp>
@@ -351,8 +361,18 @@
                 <max_vel>0.01</max_vel>
                 <min_depth>0.001</min_depth>
-              </ode>
+              </bullet>
             </contact>
           </surface>
         </collision>
+       <visual name="sphere_visual">
+          <geometry>
+            <sphere>
+              <radius>0.0060000</radius>
+            </sphere>
+          </geometry>
+          <material>
+            <diffuse>0.5 0.5 0.5</diffuse>
+          </material>
+        </visual>
       </link>
       <link name="camera_link">
